File: board/dmx_schield.sch (KiCad schematic (older format))
At the start: 48 parts, among them J1 Screw_Terminal_01x04, J2 Screw_Terminal_01x02, J3 Screw_Terminal_01x03, Q1 BC547/BSR14, SW1 SW_Push, U1 R-78E5.0-0.5, U2 MAX481E, U3 LM75B, U4 74LVC2G34

Commit message: updated board (V1.1), improved readme
Parts:
- removed Q1: BC547/BSR14, Package_TO_SOT_SMD:SOT-23, symbol Transistor_BJT:BC547
- added Q1: BSR14, Package_TO_SOT_SMD:SOT-23, symbol Device:Q_NPN_BEC
- D1, D2, D3: value LL 5819 -> BAS85; footprint Diode_SMD:D_MELF -> Diode_SMD:D_MicroMELF
Other:
- note added: "16.04.2019"
- note added: "V1.1"
Changed lines of the file:
@@
 EESchema Schematic File Version 4
-LIBS:dmx_schield-cache
 EELAYER 26 0
 EELAYER END
@@
 CLK
 $Comp
-L Transistor_BJT:BC547 Q1
-U 1 1 5D0CBE84
-P 1750 7150
-F 0 "Q1" H 1940 7196 50  0000 L CNN
-F 1 "BC547/BSR14" H 1940 7105 50  0000 L CNN
-F 2 "Package_TO_SOT_SMD:SOT-23" H 1950 7075 50  0001 L CIN
-F 3 "http://www.fairchildsemi.com/ds/BC/BC547.pdf" H 1750 7150 50  0001 L CNN
-	1    1750 7150
-	-1   0    0    -1
-$EndComp
-$Comp
 L Device:R R2
 U 1 1 5D0CC0BD
@@
 P 6850 5650
 F 0 "D2" V 6804 5571 50  0000 R CNN
-F 1 "LL 5819" V 6895 5571 50  0000 R CNN
-F 2 "Diode_SMD:D_MELF" H 6850 5650 50  0001 C CNN
+F 1 "BAS85" V 6895 5571 50  0000 R CNN
+F 2 "Diode_SMD:D_MicroMELF" H 6850 5650 50  0001 C CNN
 F 3 "~" H 6850 5650 50  0001 C CNN
 	1    6850 5650
@@
 P 7000 5950
 F 0 "D3" V 7046 6029 50  0000 L CNN
-F 1 "LL 5819" V 6955 6029 50  0000 L CNN
-F 2 "Diode_SMD:D_MELF" H 7000 5950 50  0001 C CNN
+F 1 "BAS85" V 6955 6029 50  0000 L CNN
+F 2 "Diode_SMD:D_MicroMELF" H 7000 5950 50  0001 C CNN
 F 3 "~" H 7000 5950 50  0001 C CNN
 	1    7000 5950
@@
 P 6700 5050
 F 0 "D1" V 6654 4971 50  0000 R CNN
-F 1 "LL 5819" V 6745 4971 50  0000 R CNN
-F 2 "Diode_SMD:D_MELF" H 6700 5050 50  0001 C CNN
+F 1 "BAS85" V 6745 4971 50  0000 R CNN
+F 2 "Diode_SMD:D_MicroMELF" H 6700 5050 50  0001 C CNN
 F 3 "~" H 6700 5050 50  0001 C CNN
 	1    6700 5050
@@
 Wire Wire Line
 	9900 1000 10150 1000
+$Comp
+L Device:Q_NPN_BEC Q1
+U 1 1 5D2AB6DD
+P 1750 7150
+F 0 "Q1" H 1940 7196 50  0000 L CNN
+F 1 "BSR14" H 1940 7105 50  0000 L CNN
+F 2 "Package_TO_SOT_SMD:SOT-23" H 1950 7250 50  0001 C CNN
+F 3 "~" H 1750 7150 50  0001 C CNN
+	1    1750 7150
+	-1   0    0    -1
+$EndComp
+Text Notes 8150 7650 0    50   ~ 0
+16.04.2019
+Text Notes 10600 7650 0    50   ~ 0
+V1.1
 $EndSCHEMATC

Commit message: extended and isolated  V1.0
added isolation to all elements connected to the outside world.
PCB is now a multi purpose board with as many pins as possible
available via the PCB.

I'm not happy with the PWM output stage and the connector size.
This may be changed.
Parts:
- removed D10, D5, D9: LED, LED_SMD:LED_0805_2012Metric, symbol Device:LED
- removed D4: 1N4001, Diode_SMD:D_MELF, symbol Device:D
- removed J1: Screw_Terminal_01x04, TerminalBlock_MetzConnect:TerminalBlock_MetzConnect_Type086_RT03404HBLC_1x04_P3.81mm_Horizontal, symbol Connector:Screw_Terminal_01x04
- removed J2: Screw_Terminal_01x02, TerminalBlock_MetzConnect:TerminalBlock_MetzConnect_Type086_RT03402HBLC_1x02_P3.81mm_Horizontal, symbol Connector:Screw_Terminal_01x02
- removed J3: Screw_Terminal_01x03, TerminalBlock_MetzConnect:TerminalBlock_MetzConnect_Type086_RT03403HBLC_1x03_P3.81mm_Horizontal, symbol Connector:Screw_Terminal_01x03
- removed R13, R15, R18: 100, Resistor_SMD:R_0805_2012Metric, symbol Device:R
- removed R3: 56, Resistor_SMD:R_0805_2012Metric, symbol Device:R
- removed U1: R-78E5.0-0.5, Converter_DCDC:Converter_DCDC_RECOM_R-78E-0.5_THT, symbol Regulator_Switching:R-78E5.0-0.5
- removed U3: LM75B, Package_SO:SOIC-8_3.9x4.9mm_P1.27mm, symbol Sensor_Temperature:LM75B
- added C4: 1u, Capacitor_SMD:C_0805_2012Metric, symbol Device:C
- added C50: 4,7uF/50V, Capacitor_SMD:C_1206_3216Metric, symbol Device:C
- added C51: 2,2uF/50V, Capacitor_SMD:C_1206_3216Metric, symbol Device:C
- added C6, C60: 0,1uF, Capacitor_SMD:C_0805_2012Metric, symbol Device:C
- added C61: 10uF, Capacitor_SMD:C_1206_3216Metric, symbol Device:C
- added D20, D21, D22, D23: LG R971, LED_SMD:LED_0805_2012Metric, symbol Device:LED
- added D4: BAS85, Diode_SMD:D_MicroMELF, symbol Device:D_Schottky
- added D50: TZM15, Diode_SMD:D_SC-80, symbol Device:D_Zener
- added J1, J2: Conn_01x17, Connector_PinSocket_2.54mm:PinSocket_1x17_P2.54mm_Vertical, symbol Connector_Generic:Conn_01x17
- added J250, J251: Conn_01x01, Connector_Wire:SolderWirePad_1x01_Drill0.8mm, symbol Connector_Generic:Conn_01x01
- added J30: Conn_01x04, Connector_Phoenix_MC:PhoenixContact_MC_1,5_4-G-3.81_1x04_P3.81mm_Horizontal, symbol Connector_Generic:Conn_01x04
- added J40: Conn_01x06, Connector_Phoenix_MC:PhoenixContact_MC_1,5_6-G-3.81_1x06_P3.81mm_Horizontal, symbol Connector_Generic:Conn_01x06
- added J50: Conn_01x02, Connector_Phoenix_MC:PhoenixContact_MC_1,5_2-G-3.81_1x02_P3.81mm_Horizontal, symbol Connector_Generic:Conn_01x02
- added J60: Conn_01x03, Connector_Phoenix_MC:PhoenixContact_MC_1,5_3-G-3.81_1x03_P3.81mm_Horizontal, symbol Connector_Generic:Conn_01x03
- added JP1, JP2: SolderJumper_2_Open, Jumper:SolderJumper-2_P1.3mm_Open_RoundedPad1.0x1.5mm, symbol Jumper:SolderJumper_2_Open
- added L50: 4,7uH/1.15A, Inductor_SMD:L_Bourns-SRN4018, symbol Device:L
- added Q50: IRLML5203, Package_TO_SOT_SMD:SOT-23, symbol Device:Q_PMOS_GSD
- added R130, R131, R140, R141, R260, R261, R262, R263, R264: 0, Resistor_SMD:R_0805_2012Metric, symbol Device:R
- added R142: 240, Resistor_SMD:R_0805_2012Metric, symbol Device:R
- added R143: e.g. 2k, Resistor_SMD:R_0805_2012Metric, symbol Device:R
- added R20, R21, R22, R23: 300, Resistor_SMD:R_0805_2012Metric, symbol Device:R
- added R30, R31: 540@12V, Resistor_SMD:R_0805_2012Metric, symbol Device:R
- added R4, R40, R41, R42, R43, R9: 10k, Resistor_SMD:R_0805_2012Metric, symbol Device:R
- added R50: 100k, Resistor_SMD:R_0805_2012Metric, symbol Device:R
- added R61, R62: 562, Resistor_SMD:R_0805_2012Metric, symbol Device:R
- added R8: 1,0k, Resistor_SMD:R_0805_2012Metric, symbol Device:R
- added SW2, SW3, SW4: SW_Push, Button_Switch_SMD:SW_SPST_PTS645, symbol Switch:SW_Push
- added U1: TEC 2-2411WI, my_lib:SIP8-1-2-3-5-6-7-8, symbol my_lib:DCDC-SIP8-1-2-(3)-6-7
- added U11: DCDC-SIP7-1-2-4-6, my_lib:SIP7-1-2-4-6, symbol my_lib:DCDC-SIP7-1-2-4-6
- added U140: LM317_3PinPackage, Package_TO_SOT_SMD:SOT-223-3_TabPin2, symbol Regulator_Linear:LM317_3PinPackage
- added U3: LTV-847S, Package_DIP:SMDIP-16_W7.62mm, symbol Isolator:LTV-847S
- added U5: LTV-827S, Package_DIP:SMDIP-8_W7.62mm, symbol Isolator:LTV-827S
- added U6: ADUM1301, Package_SO:SOIC-16W_7.5x10.3mm_P1.27mm, symbol my_lib:ADUM1301
- added U7: REE-0505S/1S7E_0505S1.5UP, my_lib:SIP7-1-2-4-6, symbol my_lib:DCDC-SIP7-1-2-4-6
- D6: value LED -> LH R974
- D60: renamed from D8; value LED -> LG R971
- D61: renamed from D7; value LED -> LG R971
- R10, R11: value 4,7k -> 5-10k
- R12: renamed from R1; value 56 -> 10
- R14: value 100 -> 330
- R63: renamed from R17; value 100 -> 300
- R64: renamed from R16; value 100 -> 300
- SW1: footprint Button_Switch_THT:SW_PUSH_6mm_H5mm -> Button_Switch_SMD:SW_SPST_PTS645
- U60: renamed from U2; footprint Package_DIP:DIP-8_W7.62mm -> Package_SO:PowerIntegrations_SO-8
- U61: renamed from U4; symbol 74xGxx:74LVC2G34 -> my_lib:74LVC2G34
- renumbered C3 to C1, C1 to C3, R7 to R1, R2 to R13, R9 to R2, R8 to R3, R4 to R5, R5 to R6, R12 to R60, R6 to R7, RV2 to RV1, RV1 to RV2
Connections:
- net labels added: +XV, -XV, 3V3, 3_GND, 3_VCC, 4_GND, 4_VDD, 6_GND, A2_SW1, A3_SW4, AREF, BLED, D13, DMX+, DMX-, I_PWM1, I_PWM2, I_PWM3, I_PWM4, I_SW_DOWN, I_SW_UP, MISO, POT1, POT2, PWM1, PWM2, PWM3, PWM4, RST1, RST2, RX, SCK, SCL, SDA, SW1, SW2, SW2_UP, SW3, SW3_DOWN, SW4, TX, VIN
- net labels removed: CLK, LED, POTI_KW, POTI_WW, SW_COL, SW_KW, SW_WW
- wire segments 211 -> 461
- no-connect marks 14 -> 5
Other:
- note added: "01.05.2020"
- note added: "Annotation Numbers:\n\n01-29 Main Circuit\n30-39 Button In (isolated)\n40-49 PWM Out (isolated)\n50-59 Power In (isolated)\n60-69 DMX In/Out (isolated)\n100+ Power Bridge (VIN) for isolated circuits\n200+ dangerous, bridging DMX isolation\n"
- note added: "Estimated Current @5V \n20 Arduino\n 1 LCD Dsiplay\n 40 LCD Background Amber\n100 DCDC 5V5V (+MAX481)\n100 LEDs (5x20mA)\n 2 ADUM1301\n120 Optocopler (6x20mA)\n--------------------\n\n383 Summe"
- note added: "Operating Modes\nA (resistors): Digital Output (PWM)\nB (no resistors): Low-Side Switch"
- note added: "SIL7 and SIL8 Footprints\n\nAllows to use DCDC Converter\nwith either DIL7 or DIL8 footprint\nfor more flexibilty.\n(causes Errors in Eeschema and Pcbnew)"
- note added: "V2.0"
- note added: "min out current typ/max: 3.5/10 mA\nV_O=1.25V(1+R45/R44), R44=240\n"
- note removed: "16.04.2019"
- note removed: "V1.1"
- moved on the sheet: C1, C2, C3, D3, D6, D60, D61, H1, H2, H3, H4, LCD1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
