File: board/dmx_schield.sch (KiCad schematic (older format))
At the start: 96 parts, among them J1 Conn_01x17, J2 Conn_01x17, J250 Conn_01x01, J251 Conn_01x01, J30 Conn_01x04, J40 Conn_01x06, J50 Conn_01x02, J60 Conn_01x03, Q1 BSR14, Q50 IRLML5203, SW1 SW_Push, SW2 SW_Push, SW3 SW_Push, SW4 SW_Push, U1 TEC 2-2411WI, U11 DCDC-SIP7-1-2-4-6, U140 LM317_3PinPackage, U3 LTV-847S, U5 LTV-827S, U6 ADUM1301, U60 MAX481E, U61 74LVC2G34, U7 REE-0505S/1S7E_0505S1.5UP

Commit message: fixed footprint SIL7, minor improvements, updated doc
fixed wrong pinout of SIL7 footprints and improved genral bnoard
layout and silk layer. Completed description of hardware. Added
a ods with the article numbers of the parts ordered @ reichelt.de.

This PCB verision will be manufactured and unploaded to aisler.net.
Parts:
- added C5: 10uF, Capacitor_SMD:C_1206_3216Metric, symbol Device:C
- added J41, J42, J43: Conn_01x01, Connector_Wire:SolderWirePad_1x01_Drill0.8mm, symbol Connector_Generic:Conn_01x01
- added JP40, JP41, JP42: SolderJumper_2_Bridged, Jumper:SolderJumper-2_P1.3mm_Bridged_Pad1.0x1.5mm, symbol Jumper:SolderJumper_2_Bridged
- JP1, JP2: footprint Jumper:SolderJumper-2_P1.3mm_Open_RoundedPad1.0x1.5mm -> Jumper:SolderJumper-2_P1.3mm_Open_Pad1.0x1.5mm
- LCD1: footprint my_LCD:EA DOGM 162 -> my_lib:EA_DOGM_162
- R30, R31: value 540@12V -> 560@12V
- R61, R62: value 562 -> 560
- U1: value TEC 2-2411WI -> DCDC-SIP8-1-2-(3)-6-7
Connections:
- net GND: now also C5.1
- net VCC: now also C5.2
- net 60_VCC: now reaches C60.1, C61.2, R264.1, R61.1, R63.1, R64.1, U6.10 (VE2), U6.16 (VDD2), U60.8 (VCC), U61.2 (GND), U7.6 (VOUT+)
- net 3_GND renamed 30_GND
- net 3_VCC renamed 30_VCC
- removed net 4_GND: J40.6 (Pin_6), R141.1, U3.11, U3.13, U3.15, U3.9
- net 4_VDD renamed 40_VDD
- net 40_VDD: now also J40.6 (Pin_6); no longer J40.1 (Pin_1)
- net 6_GND renamed 60_GND
- net I_SW_DOWN renamed I_SW3_DOWN
- net I_SW_UP renamed I_SW2_UP
- new net: J41.1 (Pin_1), JP40.1 (A), U3.15
- new net: J42.1 (Pin_1), JP40.2 (B), JP41.1 (A), U3.13
- new net: J43.1 (Pin_1), JP41.2 (B), JP42.1 (A), U3.11
- new net 40_GND: J40.1 (Pin_1), JP42.2 (B), R141.1, U3.9
Other:
- note added: "03.05.2020"
- note added: "Estimated Current @5V \n020 Arduino\n001 LCD Dsiplay\n040 LCD Background Amber\n100 DCDC 5V5V (+MAX481)\n100 LEDs (5x20mA)\n002 ADUM1301\n120 Optocopler (6x20mA)\n--------------------\n383 Sum"
- note added: "Home-DMX-Control"
- note removed: "01.05.2020"
- note removed: "Estimated Current @5V \n20 Arduino\n 1 LCD Dsiplay\n 40 LCD Background Amber\n100 DCDC 5V5V (+MAX481)\n100 LEDs (5x20mA)\n 2 ADUM1301\n120 Optocopler (6x20mA)\n--------------------\n\n383 Summe"
- moved on the sheet: C60, C61, D6, H1, H2, H3, H4, J250, J60, LCD1, Q1, R10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
